File: 001.brd (EAGLE design)
At the start: 100 x 80 mm, 13 parts, among them X1 0446200002, X2 0446200002, X3 0446200002, X4 0446200002

Commit message: リレーコイル電源を5V化する必要が有る場合にはレギュレータを入れる
Parts:
- added C1: 35V/2200uF, rcl:E7,5-16
- added D1: 1N4007, Diodes:DO-41
- added R1: 4.7k, rcl:0207/5V
- added U$10: (no value), Toshiba-TLP222AF:TOSHIBA_TLP222A_F_0
- added U$11: 02-JST-A, holly:B02B-XH
Connections:
- new net N$13: C1.+, D1.C, R1.2
- new net N$14: D1.A, U$11.P$1
- new net N$15: C1.-, U$10.2, U$11.P$2
- new net VCC_PD: U$10.4, U$4.2, U$7.2, X3.4, X3.5
- net N$10: now also U$3.P$1; no longer U$3.P$2
- net N$12: now also R1.1, U$10.1; no longer U$9.P$3, U$9.P$4
- net N$5: now also U$10.3, U$9.P$3; no longer U$3.P$1, U$4.2, X3.4, X3.5
- net N$6: now also U$3.P$2, U$9.P$4; no longer U$7.2
Changed lines of the file:
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@@
 <attribute name="VALUE" x="-96.52" y="-13.97" size="1.27" layer="21"/>
+</element>
+<element name="U$10" library="Toshiba-TLP222AF" package="TOSHIBA_TLP222A_F_0" value="" x="-97.79" y="-20.32" smashed="yes">
+<attribute name="NAME" x="-102.275" y="-17.43" size="1" layer="25"/>
+</element>
+<element name="C1" library="rcl" library_urn="urn:adsk.eagle:library:334" package="E7,5-16" package3d_urn="urn:adsk.eagle:package:23382/2" value="35V/2200uF" x="-95.25" y="-31.75" smashed="yes">
+<attribute name="NAME" x="-87.376" y="-27.94" size="1.778" layer="25" ratio="10"/>
+<attribute name="POPULARITY" value="4" x="-95.25" y="-31.75" size="1.778" layer="27" display="off"/>
+<attribute name="SPICEPREFIX" value="C" x="-95.25" y="-31.75" size="1.778" layer="27" display="off"/>
+<attribute name="VALUE" x="-100.33" y="-36.0426" size="1.778" layer="27" ratio="10"/>
+</element>
+<element name="D1" library="Diodes" library_urn="urn:adsk.eagle:library:11396254" package="DO-41" package3d_urn="urn:adsk.eagle:package:10898391/4" value="1N4007" x="-97.79" y="-44.45" smashed="yes">
+<attribute name="CREATED_BY" value="PCBLayout.com" x="-97.79" y="-44.45" size="1.778" layer="27" display="off"/>
+<attribute name="DIGIKEY_PART_NUMBER" value="1N4007MSCT-ND" x="-97.79" y="-44.45" size="1.778" layer="27" display="off"/>
+<attribute name="MANUFACTURER" value="Micro Commercial Co" x="-97.79" y="-44.45" size="1.778" layer="27" display="off"/>
+<attribute name="MPN" value="1N4007" x="-97.79" y="-44.45" size="1.778" layer="27" display="off"/>
+<attribute name="NAME" x="-103.29" y="-42.7" size="1.27" layer="25" ratio="10"/>
+<attribute name="PACKAGE" value="DO-41" x="-97.79" y="-44.45" size="1.778" layer="27" display="off"/>
+<attribute name="VALUE" x="-103.29" y="-47.45" size="1.27" layer="27" ratio="10"/>
+</element>
+<element name="U$11" library="holly" package="B02B-XH" value="02-JST-A" x="-109.22" y="-43.18" smashed="yes">
+<attribute name="NAME" x="-111.76" y="-39.37" size="1.27" layer="21"/>
+<attribute name="VALUE" x="-111.76" y="-46.99" size="1.27" layer="21"/>
+</element>
+<element name="R1" library="rcl" library_urn="urn:adsk.eagle:library:334" package="0207/5V" package3d_urn="urn:adsk.eagle:package:23502/1" value="4.7k" x="-109.22" y="-50.8" smashed="yes">
+<attribute name="NAME" x="-110.363" y="-49.911" size="1.27" layer="25" ratio="10"/>
+<attribute name="POPULARITY" value="0" x="-109.22" y="-50.8" size="1.778" layer="27" display="off"/>
+<attribute name="SPICEPREFIX" value="R" x="-109.22" y="-50.8" size="1.778" layer="27" display="off"/>
+<attribute name="VALUE" x="-110.363" y="-52.959" size="1.27" layer="27" ratio="10"/>
 </element>
 </elements>
@@
 <wire x1="-24.384" y1="44.958" x2="-24.384" y2="62.738" width="0" layer="19" extent="1-1"/>
 </signal>
-<signal name="N$5">
+<signal name="VCC_PD">
 <contactref element="X3" pad="4"/>
 <contactref element="X3" pad="5"/>
-<contactref element="U$3" pad="P$1"/>
 <contactref element="U$4" pad="2"/>
-<wire x1="-52.07" y1="-5.08" x2="-60.96" y2="5.08" width="0" layer="19" extent="1-1"/>
-<wire x1="-23.368" y1="43.18" x2="-60.96" y2="5.08" width="0" layer="19" extent="1-1"/>
+<contactref element="U$7" pad="2"/>
+<contactref element="U$10" pad="4"/>
+<wire x1="-53.34" y1="-12.7" x2="-93.98" y2="-19.05" width="0" layer="19" extent="1-1"/>
+<wire x1="-52.07" y1="-5.08" x2="-53.34" y2="-12.7" width="0" layer="19" extent="1-1"/>
+<wire x1="-23.368" y1="43.18" x2="-52.07" y2="-5.08" width="0" layer="19" extent="1-1"/>
 <wire x1="-22.352" y1="44.958" x2="-23.368" y2="43.18" width="0" layer="19" extent="1-1"/>
 </signal>
@@
 <contactref element="X3" pad="8"/>
 <contactref element="X3" pad="7"/>
-<contactref element="U$7" pad="2"/>
 <contactref element="U$4" pad="1"/>
-<wire x1="-59.69" y1="-5.08" x2="-53.34" y2="-12.7" width="0" layer="19" extent="1-1"/>
-<wire x1="-25.4" y1="43.18" x2="-59.69" y2="-5.08" width="0" layer="19" extent="1-1"/>
+<contactref element="U$3" pad="P$2"/>
+<contactref element="U$9" pad="P$4"/>
+<wire x1="-59.69" y1="-5.08" x2="-99.47" y2="-9.43" width="0" layer="19" extent="1-1"/>
+<wire x1="-58.42" y1="5.08" x2="-59.69" y2="-5.08" width="0" layer="19" extent="1-1"/>
+<wire x1="-25.4" y1="43.18" x2="-58.42" y2="5.08" width="0" layer="19" extent="1-1"/>
 <wire x1="-26.416" y1="44.958" x2="-25.4" y2="43.18" width="0" layer="19" extent="1-1"/>
 </signal>
@@
 <signal name="N$10">
 <contactref element="U$9" pad="P$1"/>
-<contactref element="U$3" pad="P$2"/>
-<wire x1="-58.42" y1="5.08" x2="-87.27" y2="2.57" width="0" layer="19" extent="1-1"/>
+<contactref element="U$3" pad="P$1"/>
+<wire x1="-60.96" y1="5.08" x2="-87.27" y2="2.57" width="0" layer="19" extent="1-1"/>
 </signal>
 <signal name="N$11">
@@
 <wire x1="11.02" y1="33.75" x2="11.02" y2="45.75" width="0" layer="19" extent="1-1"/>
 </signal>
+<signal name="N$5">
+<contactref element="U$10" pad="3"/>
+<contactref element="U$9" pad="P$3"/>
+<wire x1="-99.47" y1="2.57" x2="-93.98" y2="-21.59" width="0" layer="19" extent="1-1"/>
+</signal>
 <signal name="N$12">
-<contactref element="U$9" pad="P$3"/>
-<contactref element="U$9" pad="P$4"/>
-<wire x1="-99.47" y1="2.57" x2="-99.47" y2="-9.43" width="0" layer="19" extent="1-1"/>
+<contactref element="U$10" pad="1"/>
+<contactref element="R1" pad="1"/>
+<wire x1="-101.6" y1="-19.05" x2="-111.76" y2="-50.8" width="0" layer="19" extent="1-1"/>
+</signal>
+<signal name="N$13">
+<contactref element="R1" pad="2"/>
+<contactref element="D1" pad="C"/>
+<contactref element="C1" pad="+"/>
+<wire x1="-102.115" y1="-44.45" x2="-106.68" y2="-50.8" width="0" layer="19" extent="1-1"/>
+<wire x1="-99.06" y1="-31.75" x2="-102.115" y2="-44.45" width="0" layer="19" extent="1-1"/>
+</signal>
+<signal name="N$14">
+<contactref element="D1" pad="A"/>
+<contactref element="U$11" pad="P$1"/>
+<wire x1="-93.465" y1="-44.45" x2="-111.76" y2="-43.18" width="0" layer="19" extent="1-1"/>
+</signal>
+<signal name="N$15">
+<contactref element="U$10" pad="2"/>
+<contactref element="U$11" pad="P$2"/>
+<contactref element="C1" pad="-"/>
+<wire x1="-91.44" y1="-31.75" x2="-109.22" y2="-43.18" width="0" layer="19" extent="1-1"/>
+<wire x1="-101.6" y1="-21.59" x2="-91.44" y2="-31.75" width="0" layer="19" extent="1-1"/>
 </signal>
 </signals>
