File: 001.sch (KiCad schematic (older format))
At the start: 25 parts, among them CN11 02-JST-A, CN12 02-JST-A, CN21 02-JST-A, CN22 02-JST-A, J11 RJ45, J12 RJ45, J21 RJ45, J22 RJ45, K11 JQC-3FF, K21 JQC-3FF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

Commit message: PSE側art work
Parts:
- removed unit 2 of CN11
- removed unit 1 of CN12
- removed unit 1 of CN21
- removed unit 1 of CN22
- added D13, D23: LED, LED_THT:LED_D3.0mm, symbol Device:LED
- added FL11, FL21: 0.1uF DDS1, HOLLY:DSS1, symbol Device:EMI_Filter_LCL
- added R12, R22: R_US, Resistor_THT:R_Axial_DIN0207_L6.3mm_D2.5mm_P10.16mm_Horizontal, symbol Device:R_US
- CN11, CN12, CN21, CN22: value 02-JST-A -> 02-XH-A; symbol 001-eagle-import:02-JST-A -> Connector_Generic:Conn_01x02
Connections:
- net at D21.2 (A): now also CN21.1 (Pin_1)
- net at C21.2, U21.2: now also CN21.2 (Pin_2); no longer CN21.P$2 (1)
- net PSE_PWR: now reaches J11.4, J11.5, K11.4, RV11.1
- net PSE_PWR: now also R12.1
- net PSE_GND: now reaches D12.2 (A), J11.7, J11.8, K11.5, RV11.2
- net PSE_GND: now also CN12.2 (Pin_2), D13.1 (K), FL11.2; no longer CN12.P$2 (1)
- net PD_GND: now reaches D22.2 (A), J21.7, J21.8, K21.2, RV21.1
- net PD_GND: now also CN22.2 (Pin_2), FL21.2, R22.2; no longer CN22.P$2 (1)
- net at K21.4: now also D23.2 (A), FL21.1
- net PD_PWR: now reaches F21.1, J21.4, J21.5, RV21.2, U21.4
- net at D11.2 (A): now also CN11.1 (Pin_1); no longer CN11.P$1 (1)
- net at C11.2, C12.2, U11.2: now also CN11.2 (Pin_2)
- net at F11.2, U11.3: now also FL11.3
- new net: CN22.1 (Pin_1), FL21.3
- new net: CN12.1 (Pin_1), FL11.1
- new net: D13.2 (A), R12.2
- new net: D23.1 (K), R22.1
Other:
- note added: "FROM PSE"
- note added: "PD CTRL"
- note added: "PD LAN"
- note added: "PD POWER"
- note added: "PD SIDE"
- note added: "PSE CTRL"
- note added: "PSE POWER"
- note added: "PSE SIDE"
- note added: "TO PD"
- moved on the sheet: C21, D21, J12, R21

Commit message: もうちょっとRJ45コネクタは大変更
Parts:
- J11, J12, J21, J22: footprint Connector_RJ:RJ45_Amphenol_RJHSE5380 -> HOLLY:RJ45_Neltron_7810-8P8C
Changed lines of the file:
@@
 F 0 "J21" H 6057 4067 50  0000 C CNN
 F 1 "RJ45" H 6057 3976 50  0000 C CNN
-F 2 "Connector_RJ:RJ45_Amphenol_RJHSE5380" V 6000 3425 50  0001 C CNN
+F 2 "HOLLY:RJ45_Neltron_7810-8P8C" V 6000 3425 50  0001 C CNN
 F 3 "~" V 6000 3425 50  0001 C CNN
 	1    6000 3400
@@
 F 0 "J22" H 7370 4804 50  0000 R CNN
 F 1 "RJ45" H 7370 4895 50  0000 R CNN
-F 2 "Connector_RJ:RJ45_Amphenol_RJHSE5380" V 7700 4825 50  0001 C CNN
+F 2 "HOLLY:RJ45_Neltron_7810-8P8C" V 7700 4825 50  0001 C CNN
 F 3 "~" V 7700 4825 50  0001 C CNN
 	1    7700 4800
@@
 F 0 "J11" H 4270 3304 50  0000 R CNN
 F 1 "RJ45" H 4270 3395 50  0000 R CNN
-F 2 "Connector_RJ:RJ45_Amphenol_RJHSE5380" V 4600 3325 50  0001 C CNN
+F 2 "HOLLY:RJ45_Neltron_7810-8P8C" V 4600 3325 50  0001 C CNN
 F 3 "~" V 4600 3325 50  0001 C CNN
 	1    4600 3300
@@
 F 0 "J12" H 3057 6367 50  0000 C CNN
 F 1 "RJ45" H 3057 6276 50  0000 C CNN
-F 2 "Connector_RJ:RJ45_Amphenol_RJHSE5380" V 3000 5725 50  0001 C CNN
+F 2 "HOLLY:RJ45_Neltron_7810-8P8C" V 3000 5725 50  0001 C CNN
 F 3 "~" V 3000 5725 50  0001 C CNN
 	1    3000 5700
@@
 Wire Wire Line
 	8700 2500 8700 2800
-Wire Bus Line
-	3850 2900 3850 6100
-Wire Bus Line
-	7000 3200 7000 5100
 Text Notes 8400 4100 0    500  ~ 0
 PD SIDE
@@
 Text Label 4000 2300 0    50   ~ 0
 PSE_PWR
+Wire Bus Line
+	3850 2900 3850 6100
+Wire Bus Line
+	7000 3200 7000 5100
 $EndSCHEMATC

Commit message: 一応完成、これからガーバー
Changed lines of the file:
@@
 Wire Bus Line
 	7000 3200 7000 5100
+Text Label 2400 3600 0    50   ~ 0
+PSE_GND
 $EndSCHEMATC

Commit message: PSEとPDを別図面にした
Parts:
- removed C11: 35V/10uF, Capacitor_THT:C_Disc_D6.0mm_W2.5mm_P5.00mm, symbol Device:CP
- removed C12: 35V/2200uF, Capacitor_THT:CP_Radial_D16.0mm_P7.50mm, symbol Device:CP
- removed CN11, CN12: 02-XH-A, Connector_JST:JST_XH_B2B-XH-A_1x02_P2.50mm_Vertical, symbol Connector_Generic:Conn_01x02
- removed D11, D12: 1N4007, Diode_THT:D_DO-41_SOD81_P10.16mm_Horizontal, symbol Diode:1N4007
- removed D13: LED, LED_THT:LED_D3.0mm, symbol Device:LED
- removed F11: LVR040, Fuse:Fuse_BelFuse_0ZRE0033FF_L11.4mm_W3.8mm, symbol Device:Polyfuse
- removed FL11: 0.1uF DDS1, HOLLY:DSS1, symbol Device:EMI_Filter_LCL
- removed J11, J12: RJ45, HOLLY:RJ45_Neltron_7810-8P8C, symbol Connector:RJ45
- removed K11: JQC-3FF, Relay_THT:Relay_SPDT_Omron-G5LE-1, symbol Relay:G5LE-1
- removed R11: 4.7k, Resistor_THT:R_Axial_DIN0207_L6.3mm_D2.5mm_P10.16mm_Horizontal, symbol Device:R_US
- removed R12: R_US, Resistor_THT:R_Axial_DIN0207_L6.3mm_D2.5mm_P10.16mm_Horizontal, symbol Device:R_US
- removed RV11: TNR10V471K, Varistor:RV_Disc_D12mm_W3.9mm_P7.5mm, symbol Device:Varistor_US
- removed U11: TLP222A, Package_DIP:DIP-4_W7.62mm, symbol Relay_SolidState:TLP222A
Connections:
- no-connect marks 11 -> 6
Other:
- note removed: "C-00159"
- note removed: "PSE CTRL"
- note removed: "PSE POWER"
- note removed: "PSE SIDE"
- note removed: "TO PD"
- moved on the sheet: C21, CN21, CN22, D21, D22, D23, F21, FL21, J21, J22, K21, R21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

Commit message: version合わせ
Parts:
- R21: value 4.7k -> 3.3k
- R22: value R_US -> 4.7k
Other:
- note removed: "Model-800\nNCxPoE"
- note removed: "PD SIDE"
Changed lines of the file:
@@
 EELAYER 30 0
 EELAYER END
-$Descr User 11774 8671
+$Descr A4 11693 8268
 encoding utf-8
 Sheet 1 1
-Title ""
-Date ""
-Rev ""
+Title "M800-NCxPoE-PD"
+Date "2020-08-08"
+Rev "001"
 Comp ""
-Comment1 ""
-Comment2 ""
+Comment1 "PD SIDE"
+Comment2 "Vcc=5V"
 Comment3 ""
 Comment4 ""
@@
 F 3 "" H 8050 2900 50  0001 C CNN
 	1    8050 2900
-	1    0    0    -1
-$EndComp
-$Comp
-L 001-eagle-import:A4L-LOC #FRAME1
-U 1 1 73DA64CA
-P 900 7100
-F 0 "#FRAME1" H 900 7100 50  0001 C CNN
-F 1 "A4L-LOC" H 900 7100 50  0001 C CNN
-F 2 "" H 900 7100 50  0001 C CNN
-F 3 "" H 900 7100 50  0001 C CNN
-	1    900  7100
 	1    0    0    -1
 $EndComp
@@
 P 7000 1200
 F 0 "R21" V 6950 1100 59  0000 L BNN
-F 1 "4.7k" V 7100 1100 59  0000 L BNN
+F 1 "3.3k" V 7100 1100 59  0000 L BNN
 F 2 "Resistor_THT:R_Axial_DIN0207_L6.3mm_D2.5mm_P10.16mm_Horizontal" H 7000 1200 50  0001 C CNN
 F 3 "" H 7000 1200 50  0001 C CNN
@@
 	0    1    1    0
 $EndComp
-Text Notes 7500 6900 0    215  ~ 0
-Model-800\nNCxPoE
 $Comp
 L Connector:RJ45 J21
@@
 U 1 1 5F0794E0
 P 6450 2700
-F 0 "R22" V 6245 2700 50  0000 C CNN
-F 1 "R_US" V 6336 2700 50  0000 C CNN
+F 0 "R22" V 6350 2700 50  0000 C CNN
+F 1 "4.7k" V 6550 2700 50  0000 C CNN
 F 2 "Resistor_THT:R_Axial_DIN0207_L6.3mm_D2.5mm_P10.16mm_Horizontal" V 6490 2690 50  0001 C CNN
 F 3 "~" H 6450 2700 50  0001 C CNN
@@
 U 1 1 5F082CA7
 P 6850 2700
-F 0 "D23" H 6843 2917 50  0000 C CNN
-F 1 "LED" H 6843 2826 50  0000 C CNN
+F 0 "D23" H 6850 2800 50  0000 C CNN
+F 1 "LED" H 6850 2600 50  0000 C CNN
 F 2 "LED_THT:LED_D3.0mm" H 6850 2700 50  0001 C CNN
 F 3 "~" H 6850 2700 50  0001 C CNN
@@
 Wire Wire Line
 	6200 2700 6200 3000
-Text Notes 5900 4300 0    500  ~ 0
-PD SIDE
 Text Notes 8150 1500 0    50   ~ 0
 PD CTRL
