File: 002.sch (KiCad schematic (older format))
At the start: 16 parts, among them CN11 02-XH-A, CN12 02-XH-A, J11 RJ45, J12 RJ45, K11 JQC-3FF, U11 TLP222A

Commit message: version合わせ
Parts:
- R11: value 4.7k -> 3.3k
- R12: value R_US -> 4.7k
Other:
- note removed: "Model-800\nNCxPoE"
- note removed: "PSE SIDE"
Changed lines of the file:
@@
 encoding utf-8
 Sheet 1 1
-Title ""
-Date ""
-Rev ""
+Title "M800-NCxPoE-PSE"
+Date "2020-08-08"
+Rev "001"
 Comp ""
-Comment1 ""
-Comment2 ""
+Comment1 "Vcc=5V"
+Comment2 "PSE SIDE"
 Comment3 ""
 Comment4 ""
@@
 $EndComp
 $Comp
-L 001-eagle-import:A4L-LOC #FRAME1
-U 1 1 73DA64CA
-P 900 7100
-F 0 "#FRAME1" H 900 7100 50  0001 C CNN
-F 1 "A4L-LOC" H 900 7100 50  0001 C CNN
-F 2 "" H 900 7100 50  0001 C CNN
-F 3 "" H 900 7100 50  0001 C CNN
-	1    900  7100
-	1    0    0    -1
-$EndComp
-$Comp
 L Relay:G5LE-1 K11
 U 1 1 E90442EA
@@
 Text Notes 6700 3300 0    59   ~ 0
 C-00159
-Text Notes 7500 6900 0    215  ~ 0
-Model-800\nNCxPoE
 $Comp
 L Connector:RJ45 J11
@@
 P 5400 1350
 F 0 "R11" V 5350 1250 59  0000 L BNN
-F 1 "4.7k" V 5500 1250 59  0000 L BNN
+F 1 "3.3k" V 5500 1250 59  0000 L BNN
 F 2 "Resistor_THT:R_Axial_DIN0207_L6.3mm_D2.5mm_P10.16mm_Horizontal" H 5400 1350 50  0001 C CNN
 F 3 "" H 5400 1350 50  0001 C CNN
@@
 P 6000 3100
 F 0 "R12" H 6068 3146 50  0000 L CNN
-F 1 "R_US" H 6068 3055 50  0000 L CNN
+F 1 "4.7k" H 6068 3055 50  0000 L CNN
 F 2 "Resistor_THT:R_Axial_DIN0207_L6.3mm_D2.5mm_P10.16mm_Horizontal" V 6040 3090 50  0001 C CNN
 F 3 "~" H 6000 3100 50  0001 C CNN
@@
 Wire Wire Line
 	6000 4100 6500 4100
-Text Notes 2650 5100 0    500  ~ 0
-PSE SIDE
 Text Notes 6900 3550 0    50   ~ 0
 TO PD
