File: 002.kicad_pcb (KiCad board)
At the start: 2 copper layers, 55.9 x 55.9 mm, 30 parts, among them CN11 02-XH-A, CN12 02-XH-A, J11 RJ45, J12 RJ45, K11 JQC-3FF, U11 TLP222A

Commit message: KiCAD Version
Parts:
- removed the ? at (85.1, 73.0) (x2)
- added ? (x2): , , F.Cu at (85.1, 73.0)
Other:
- net class Default removed
